File: pcb_sram.sch (KiCad schematic (older format))
At the start: 47 parts, among them P1 DIL32, P2 DIL32, P3 DIL32, P4 DIL32, P6 CONN_3, P7 KNUSB, P8 MICRO-SD, U1 STM32F40X_LQFP144, U2 CY62177D, U3 CY62177D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

Commit message: Add footprints for components. Various misc. small fixes.
Parts:
- C5, C6, C7: value CSMALL -> 100n
Connections:
- wire segments 538 -> 536
- no-connect marks 1 -> 2

Commit message: Couple changes to the schematics after review:
 - Full-size SD card instead of micro-SD card.

 - Power LED, user LED

 - Use 0805 instead of 0603 for capacitors.
Parts:
- removed P8: MICRO-SD, symbol MICRO-SD
- added D1: SML-211UTT86, symbol LED
- added D2: SML-211YTT86, symbol LED
- added P8: SD_CARD, symbol SD_CARD
- added R1, R2: 1k, symbol R
Connections:
- net labels added: sd_wp, user_led
- net labels removed: pc14, pg15
- wire segments 536 -> 544

Commit message: Add reset button.
Parts:
- added B1: SWITCH_4PIN, symbol SWITCH_4PIN
Connections:
- wire segments 544 -> 552
Other:
- moved on the sheet: D1, D2, R1, R2

Commit message: First partial PCB layout.
 - Move components into place

 - Hand-route the critical parts

 - Set board edge

 - Removed extra SRAM chips, lets go with just one
Parts:
- removed C5, C6, C7: 100n, symbol CSMALL
- removed U3, U4, U5: CY62177D, symbol CY62177D
Connections:
- wire segments 552 -> 402

Commit message: Rounded corners on the PCB, and connect SD card shield to ground.
Connections:
- wire segments 402 -> 404
- no-connect marks 2 -> 1
